File: hardware/mainboard/kicad/enku-mainboard-r0.1.kicad_pcb (KiCad board)
At the start: 4 copper layers, 54 x 94 mm, 122 parts, among them J1 1S LiPo + NTC, J2 Hirose DM3AT-SF-PEJM5, J3 FH34SRJ-24S-0.5SH(50), J5 GCT USB4105-GF-A-120, J6 4-pin pogo dock, J7 Tag-Connect TC2030-IDC-NL, Q1 IRLML6346TRPBF, SW1 HARD POWER, SW2 BOOT / RECOVERY, SW3 BTN_L1, SW4 BTN_L2, SW5 BTN_R1, SW6 BTN_R2, U1 ESP32-S3-WROOM-1-N16R8, U2 TPS2121, U3 BQ25185DLHR, U4 TPS63802DLAR, U5 BMI270, U6 DRV5032FBDBZR, U8 USBLC6-2SC6

Commit message: pcb: move BTN_R2 trunk off USB corridor
Routing:
- net BTN_R2: track 54.9 -> 57.9 mm, vias 2 -> 4
Changed lines of the file:
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@@
   (segment (start 69.00 60.80) (end 71.20 60.80) (width 0.18) (layer "F.Cu") (net 50))
   (segment (start 35.36 53.75) (end 35.36 56.00) (width 0.18) (layer "F.Cu") (net 51))
-  (via (at 35.36 56.00) (size 0.60) (drill 0.30) (layers "F.Cu" "In2.Cu") (net 51))
-  (segment (start 35.36 56.00) (end 66.20 56.00) (width 0.18) (layer "In2.Cu") (net 51))
-  (segment (start 66.20 72.80) (end 68.00 72.80) (width 0.18) (layer "In2.Cu") (net 51))
-  (via (at 68.00 72.80) (size 0.60) (drill 0.30) (layers "F.Cu" "In2.Cu") (net 51))
+  (via (at 35.36 56.00) (size 0.60) (drill 0.30) (layers "F.Cu" "B.Cu") (net 51))
+  (via (at 68.00 72.80) (size 0.60) (drill 0.30) (layers "F.Cu" "B.Cu") (net 51))
   (segment (start 68.00 72.80) (end 71.20 72.80) (width 0.18) (layer "F.Cu") (net 51))
   (segment (start 45.0 87.2) (end 49.8 87.2) (width 0.18) (layer "In2.Cu") (net 90))
@@
   (segment (start 34.000 89.200) (end 36.270 89.200) (width 0.18) (layer "B.Cu") (net 47))
   (segment (start 36.270 89.200) (end 36.270 87.635) (width 0.18) (layer "B.Cu") (net 47))
-  (segment (start 66.20 56.00) (end 66.20 72.80) (width 0.18) (layer "In2.Cu") (net 51))
   (segment (start 29.010 34.000) (end 22.000 50.000) (width 0.18) (layer "In2.Cu") (net 73))
   (segment (start 30.280 34.000) (end 23.000 45.000) (width 0.18) (layer "In2.Cu") (net 72))
@@
   (segment (start 67.00 54.00) (end 67.00 60.80) (width 0.18) (layer "B.Cu") (net 50))
   (segment (start 67.00 60.80) (end 69.00 60.80) (width 0.18) (layer "B.Cu") (net 50))
+  (segment (start 35.36 56.00) (end 35.36 54.50) (width 0.18) (layer "B.Cu") (net 51))
+  (segment (start 35.36 54.50) (end 37.40 54.50) (width 0.18) (layer "B.Cu") (net 51))
+  (via (at 37.40 54.50) (size 0.45) (drill 0.20) (layers "B.Cu" "In1.Cu") (net 51))
+  (segment (start 37.40 54.50) (end 38.60 54.50) (width 0.18) (layer "In1.Cu") (net 51))
+  (via (at 38.60 54.50) (size 0.45) (drill 0.20) (layers "B.Cu" "In1.Cu") (net 51))
+  (segment (start 38.60 54.50) (end 66.20 54.50) (width 0.18) (layer "B.Cu") (net 51))
+  (segment (start 66.20 54.50) (end 66.20 72.80) (width 0.18) (layer "B.Cu") (net 51))
+  (segment (start 66.20 72.80) (end 68.00 72.80) (width 0.18) (layer "B.Cu") (net 51))
 )
