File: hardware/mainboard/kicad/enku-mainboard-r0.7-base-dfm-prep.kicad_pcb (KiCad board)
At the start: 4 copper layers, 59 x 101 mm, 120 parts, among them J1 1S LiPo + NTC, J2 Hirose DM3AT-SF-PEJM5, J3 FH34SRJ-24S-0.5SH(50), J5 GCT USB4105-GF-A-120, J6 4-pin pogo dock, J7 TC2030-IDC-NL / DNL, Q1 IRLML6346TRPBF, SW1 HARD POWER, SW2 BOOT / RECOVERY, SW3 BTN_L1, SW4 BTN_L2, SW5 BTN_R1, SW6 BTN_R2, U1 ESP32-S3-WROOM-1-N16R8, U2 TPS2121, U3 BQ25185DLHR, U4 TPS63802DLAR, U5 BMI270, U8 USBLC6-2SC6

Commit message: R30: align J6 bare contact BOM and J7 service header value with schematic
Parts:
- J7: value TC2030-IDC-NL / DNL -> Tag-Connect TC2030-IDC-NL
Changed lines of the file:
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@@
     (at 35 87)
     (property "Reference" "J7" (at 0 2.7 0) (layer "B.SilkS"))
-    (property "Value" "TC2030-IDC-NL / DNL" (at 0 -2.3 0) (layer "B.Fab") hide)
+    (property "Value" "Tag-Connect TC2030-IDC-NL" (at 0 -2.3 0) (layer "B.Fab") hide)
     (attr exclude_from_bom exclude_from_pos_files)
     (fp_rect (start -3.5 -2) (end 3.5 2) (stroke (width 0.05) (type default)) (fill none) (layer "B.CrtYd"))
