File: hardware/mainboard/kicad/mcu_io.kicad_sch (KiCad schematic)
At the start: 37 parts, among them J2 Hirose DM3AT-SF-PEJM5, SW2 BOOT / RECOVERY, SW3 BTN_L1, SW4 BTN_L2, SW5 BTN_R1, SW6 BTN_R2, U1 ESP32-S3-WROOM-1-N16R8, U10 TLV3012BIDBVR, U5 BMI270, U9 TMUX1101DBVR

Commit message: hardware: preserve recovered R119 layout and verified R118 source [skip ci]
Persist the KiCad 10.0.7 project before the next routing pass. The recovered layout has 67 opens, ERC 0, parity 0 and zero RF keepout violations; routing is incomplete and fabrication is blocked. Preserve all pad and surviving copper net identities and retain an immutable R118 source archive.
Parts:
- SW3: value BTN_L1 -> TL3340AF160QG; footprint ENKU:READING_BUTTON_PLACEMENT -> ENKU:TL3340AF160QG_GEOMETRY_TRIAL; symbol ENKU:SW -> ENKU:TL3340_3PIN
- SW4: value BTN_L2 -> TL3340AF160QG; footprint ENKU:READING_BUTTON_PLACEMENT -> ENKU:TL3340AF160QG_GEOMETRY_TRIAL; symbol ENKU:SW -> ENKU:TL3340_3PIN
- SW5: value BTN_R1 -> TL3340AF160QG; footprint ENKU:READING_BUTTON_PLACEMENT -> ENKU:TL3340AF160QG_GEOMETRY_TRIAL; symbol ENKU:SW -> ENKU:TL3340_3PIN
- SW6: value BTN_R2 -> TL3340AF160QG; footprint ENKU:READING_BUTTON_PLACEMENT -> ENKU:TL3340AF160QG_GEOMETRY_TRIAL; symbol ENKU:SW -> ENKU:TL3340_3PIN
Connections:
- net GND: now also SW3.3 (B), SW4.3 (B), SW5.3 (B), SW6.3 (B); no longer SW3.2 (B), SW4.2 (B), SW5.2 (B), SW6.2 (B)
- net DOCK_DETECT: no longer names the net of U1.38 (GPIO2)
- no-connect marks 19 -> 20
Changed lines of the file:
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@@
 	(global_label "UART_RX" (shape output) (at 104.14 97.79 180) (effects (font (size 0.88 0.88)) (justify right bottom)))
 	(global_label "UART_TX" (shape output) (at 104.14 100.33 180) (effects (font (size 0.88 0.88)) (justify right bottom)))
-	(global_label "DOCK_DETECT" (shape output) (at 104.14 102.87 180) (effects (font (size 0.88 0.88)) (justify right bottom)))
+	(no_connect (at 104.14 102.87))
 	(global_label "BAT_ADC" (shape output) (at 104.14 105.41 180) (effects (font (size 0.88 0.88)) (justify right bottom)))
 	(no_connect (at 60.96 93.98))
@@
 	(global_label "BOOT" (shape input) (at 123.19 132.08 0) (effects (font (size 0.88 0.88)) (justify right bottom)))
 	(global_label "GND" (shape output) (at 139.7 132.08 180) (effects (font (size 0.88 0.88)) (justify right bottom)))
-	(symbol (lib_id "ENKU:SW") (at 32.385 166.37 0) (unit 1) (exclude_from_sim no) (in_bom yes) (on_board yes) (dnp no)
+	(symbol (lib_id "ENKU:TL3340_3PIN") (at 32.385 166.37 0) (unit 1) (exclude_from_sim no) (in_bom yes) (on_board yes) (dnp no)
 		(property "Reference" "SW3" (at 26.385 149.37 0) (effects (font (size 0.88 0.88))))
-		(property "Value" "BTN_L1" (at 38.385 149.37 0) (effects (font (size 0.88 0.88))))
-		(property "Footprint" "ENKU:READING_BUTTON_PLACEMENT" (at 32.385 166.37 0) (effects (font (size 0.88 0.88)) (hide yes)))
+		(property "Value" "TL3340AF160QG" (at 38.385 149.37 0) (effects (font (size 0.88 0.88))))
+		(property "Footprint" "ENKU:TL3340AF160QG_GEOMETRY_TRIAL" (at 32.385 166.37 0) (effects (font (size 0.88 0.88)) (hide yes)))
 		(property "Datasheet" "~" (at 32.385 166.37 0) (effects (font (size 0.88 0.88)) (hide yes)))
 		(property "Description" "BTN_L1" (at 32.385 166.37 0) (effects (font (size 0.88 0.88)) (hide yes)))
 		(pin "1")
-		(pin "2")
+		(pin "3")
 		(instances (project "enku-mainboard-r0.1" (path "/10000000-0000-4000-8000-000000000001/74000000-0000-4000-8000-000000000110" (reference "SW3") (unit 1))))
 	)
 	(global_label "BTN_L1" (shape input) (at 24.13 166.37 0) (effects (font (size 0.88 0.88)) (justify right bottom)))
 	(global_label "GND" (shape output) (at 40.64 166.37 180) (effects (font (size 0.88 0.88)) (justify right bottom)))
-	(symbol (lib_id "ENKU:SW") (at 61.595 166.37 0) (unit 1) (exclude_from_sim no) (in_bom yes) (on_board yes) (dnp no)
+	(symbol (lib_id "ENKU:TL3340_3PIN") (at 61.595 166.37 0) (unit 1) (exclude_from_sim no) (in_bom yes) (on_board yes) (dnp no)
 		(property "Reference" "SW4" (at 55.595 149.37 0) (effects (font (size 0.88 0.88))))
-		(property "Value" "BTN_L2" (at 67.595 149.37 0) (effects (font (size 0.88 0.88))))
-		(property "Footprint" "ENKU:READING_BUTTON_PLACEMENT" (at 61.595 166.37 0) (effects (font (size 0.88 0.88)) (hide yes)))
+		(property "Value" "TL3340AF160QG" (at 67.595 149.37 0) (effects (font (size 0.88 0.88))))
+		(property "Footprint" "ENKU:TL3340AF160QG_GEOMETRY_TRIAL" (at 61.595 166.37 0) (effects (font (size 0.88 0.88)) (hide yes)))
 		(property "Datasheet" "~" (at 61.595 166.37 0) (effects (font (size 0.88 0.88)) (hide yes)))
 		(property "Description" "BTN_L2" (at 61.595 166.37 0) (effects (font (size 0.88 0.88)) (hide yes)))
 		(pin "1")
-		(pin "2")
+		(pin "3")
 		(instances (project "enku-mainboard-r0.1" (path "/10000000-0000-4000-8000-000000000001/74000000-0000-4000-8000-000000000115" (reference "SW4") (unit 1))))
 	)
 	(global_label "BTN_L2" (shape input) (at 53.34 166.37 0) (effects (font (size 0.88 0.88)) (justify right bottom)))
 	(global_label "GND" (shape output) (at 69.85 166.37 180) (effects (font (size 0.88 0.88)) (justify right bottom)))
-	(symbol (lib_id "ENKU:SW") (at 92.075 166.37 0) (unit 1) (exclude_from_sim no) (in_bom yes) (on_board yes) (dnp no)
+	(symbol (lib_id "ENKU:TL3340_3PIN") (at 92.075 166.37 0) (unit 1) (exclude_from_sim no) (in_bom yes) (on_board yes) (dnp no)
 		(property "Reference" "SW5" (at 86.075 149.37 0) (effects (font (size 0.88 0.88))))
-		(property "Value" "BTN_R1" (at 98.075 149.37 0) (effects (font (size 0.88 0.88))))
-		(property "Footprint" "ENKU:READING_BUTTON_PLACEMENT" (at 92.075 166.37 0) (effects (font (size 0.88 0.88)) (hide yes)))
+		(property "Value" "TL3340AF160QG" (at 98.075 149.37 0) (effects (font (size 0.88 0.88))))
+		(property "Footprint" "ENKU:TL3340AF160QG_GEOMETRY_TRIAL" (at 92.075 166.37 0) (effects (font (size 0.88 0.88)) (hide yes)))
 		(property "Datasheet" "~" (at 92.075 166.37 0) (effects (font (size 0.88 0.88)) (hide yes)))
 		(property "Description" "BTN_R1" (at 92.075 166.37 0) (effects (font (size 0.88 0.88)) (hide yes)))
 		(pin "1")
-		(pin "2")
+		(pin "3")
 		(instances (project "enku-mainboard-r0.1" (path "/10000000-0000-4000-8000-000000000001/74000000-0000-4000-8000-000000000120" (reference "SW5") (unit 1))))
 	)
 	(global_label "BTN_R1" (shape input) (at 83.82 166.37 0) (effects (font (size 0.88 0.88)) (justify right bottom)))
 	(global_label "GND" (shape output) (at 100.33 166.37 180) (effects (font (size 0.88 0.88)) (justify right bottom)))
-	(symbol (lib_id "ENKU:SW") (at 122.555 166.37 0) (unit 1) (exclude_from_sim no) (in_bom yes) (on_board yes) (dnp no)
+	(symbol (lib_id "ENKU:TL3340_3PIN") (at 122.555 166.37 0) (unit 1) (exclude_from_sim no) (in_bom yes) (on_board yes) (dnp no)
 		(property "Reference" "SW6" (at 116.555 149.37 0) (effects (font (size 0.88 0.88))))
-		(property "Value" "BTN_R2" (at 128.555 149.37 0) (effects (font (size 0.88 0.88))))
-		(property "Footprint" "ENKU:READING_BUTTON_PLACEMENT" (at 122.555 166.37 0) (effects (font (size 0.88 0.88)) (hide yes)))
+		(property "Value" "TL3340AF160QG" (at 128.555 149.37 0) (effects (font (size 0.88 0.88))))
+		(property "Footprint" "ENKU:TL3340AF160QG_GEOMETRY_TRIAL" (at 122.555 166.37 0) (effects (font (size 0.88 0.88)) (hide yes)))
 		(property "Datasheet" "~" (at 122.555 166.37 0) (effects (font (size 0.88 0.88)) (hide yes)))
 		(property "Description" "BTN_R2" (at 122.555 166.37 0) (effects (font (size 0.88 0.88)) (hide yes)))
 		(pin "1")
-		(pin "2")
+		(pin "3")
 		(instances (project "enku-mainboard-r0.1" (path "/10000000-0000-4000-8000-000000000001/74000000-0000-4000-8000-000000000125" (reference "SW6") (unit 1))))
 	)

Commit message: hardware: R123 button and microSD geometry audit with native guards; NO FAB
Connections:
- no-connect marks 20 -> 24
Changed lines of the file:
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@@
 (global_label "USB_VBUS_DIV" (shape input) (at 359.41 261.62 0) (effects (font (size 0.88 0.88)) (justify right bottom)))
 (global_label "GND" (shape input) (at 374.65 261.62 180) (effects (font (size 0.88 0.88)) (justify right bottom)))
+	(no_connect (at 33.02 173.99))
+	(no_connect (at 62.23 173.99))
+	(no_connect (at 92.71 173.99))
+	(no_connect (at 123.19 173.99))
 )

Commit message: R125: correct manufacturer Q1/Q2/U9 lands and guard full copper, netlist and assembly layers
Parts:
- U9: footprint Package_TO_SOT_SMD:SOT-23-5 -> ENKU:TMUX1101_TI_DBV0005A
Changed lines of the file:
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@@
 (property "Reference" "U9" (at 325.2 158.6 0) (effects (font (size 0.88 0.88))))
 (property "Value" "TMUX1101DBVR" (at 335.2 158.6 0) (effects (font (size 0.88 0.88))))
-(property "Footprint" "Package_TO_SOT_SMD:SOT-23-5" (at 330.2 174.6 0) (effects (font (size 0.88 0.88)) (hide yes)))
+(property "Footprint" "ENKU:TMUX1101_TI_DBV0005A" (at 330.2 174.6 0) (effects (font (size 0.88 0.88)) (hide yes)))
 (property "Datasheet" "https://www.ti.com/lit/ds/symlink/tmux1101.pdf" (at 330.2 174.6 0) (effects (font (size 0.88 0.88)) (hide yes)))
 (property "Description" "TMUX1101DBVR" (at 330.2 174.6 0) (effects (font (size 0.88 0.88)) (hide yes)))

Commit message: R126: select 61 exact components, correct physical lands and local routing, preserve full source; NO FAB
Parts:
- C13: footprint Capacitor_SMD:C_0805_2012Metric -> ENKU:C_CC0805_YAGEO_REFLOW_TRANSFER; Assembly (none) -> FIT; MPN (none) -> CC0805KKX5R6BB106; Manufacturer (none) -> Yageo; Voltage (none) -> 10V
- C37: footprint Capacitor_SMD:C_0603_1608Metric -> ENKU:C_CC0603_YAGEO_REFLOW_TRANSFER; Assembly (none) -> FIT; MPN (none) -> CC0603KRX7R9BB104; Manufacturer (none) -> Yageo; Voltage (none) -> 50V
- R17, R18: footprint Resistor_SMD:R_0603_1608Metric -> ENKU:R_RC0603_YAGEO_REFLOW; Assembly (none) -> FIT; MPN (none) -> RC0603FR-0710KL; Manufacturer (none) -> Yageo
- R19: footprint Resistor_SMD:R_0603_1608Metric -> ENKU:R_RC0603_YAGEO_REFLOW; Assembly (none) -> FIT; MPN (none) -> RC0603JR-070RL; Manufacturer (none) -> Yageo
- R20, R21, R22: footprint Resistor_SMD:R_0603_1608Metric -> ENKU:R_RC0603_YAGEO_REFLOW; Assembly (none) -> FIT; MPN (none) -> RC0603JR-070RL; Manufacturer (none) -> Yageo; Tuning MPN (none) -> RC0603FR-0722RL
- R23: footprint Resistor_SMD:R_0603_1608Metric -> ENKU:R_RC0603_YAGEO_REFLOW; Assembly (none) -> FIT; MPN (none) -> RC0603FR-0747KL; Manufacturer (none) -> Yageo
- R24, R25: footprint Resistor_SMD:R_0603_1608Metric -> ENKU:R_RC0603_YAGEO_REFLOW; Assembly (none) -> FIT; MPN (none) -> RC0603FR-074K7L; Manufacturer (none) -> Yageo
- R26: footprint Resistor_SMD:R_0603_1608Metric -> ENKU:R_RC0603_YAGEO_REFLOW; Assembly (none) -> FIT; MPN (none) -> RC0603FR-072ML; Manufacturer (none) -> Yageo
- R27: footprint Resistor_SMD:R_0603_1608Metric -> ENKU:R_RC0603_YAGEO_REFLOW; Assembly (none) -> FIT; MPN (none) -> RC0603FR-07680KL; Manufacturer (none) -> Yageo
- R39: footprint Resistor_SMD:R_0603_1608Metric -> ENKU:R_RC0603_YAGEO_REFLOW; Assembly (none) -> FIT; MPN (none) -> RC0603FR-071ML; Manufacturer (none) -> Yageo
- R72: footprint Resistor_SMD:R_0603_1608Metric -> ENKU:R_RC0603_YAGEO_REFLOW; Assembly (none) -> FIT; MPN (none) -> RC0603FR-07100KL; Manufacturer (none) -> Yageo
- R73: footprint Resistor_SMD:R_0603_1608Metric -> ENKU:R_RC0603_YAGEO_REFLOW; Assembly (none) -> FIT; MPN (none) -> RC0603FR-073K3L; Manufacturer (none) -> Yageo
- SW2: footprint Button_Switch_SMD:SW_SPST_TL3342 -> ENKU:TL3342F160QG_ESWITCH_P010632J; Assembly (none) -> FIT; MPN (none) -> TL3342F160QG; Manufacturer (none) -> E-Switch

Commit message: R127: finish passive MPN selection and correct USB VBUS capacitance
Select exact parts and nominal lands for the remaining 15 capacitors and R70/R71/R37. Reduce C4 from10uF/10V to1uF/25V, taking direct VBUS capacitance from15.8 to6.8uF. Preserve all417 original pad and2639 Cu identities/nets, with only3 declared EPD_VCI vertex adjustments.

Native KiCad10.0.7: opens0/ERC0/parity0/DRC47(27library+20holes). Add independent79-part, source and native-netlist numeric power guards. Record unqualified Ceff, inrush, EPD pulse/process gates; NO FAB.
Parts:
- C14, C17, C18, C19, C21, C38: footprint Capacitor_SMD:C_0603_1608Metric -> ENKU:C_CC0603_YAGEO_REFLOW_TRANSFER; Assembly (none) -> FIT; MPN (none) -> CC0603KRX7R9BB104; Manufacturer (none) -> Yageo; Voltage (none) -> 50V
- C15: footprint Capacitor_SMD:C_0603_1608Metric -> ENKU:C_CC0603_YAGEO_REFLOW_TRANSFER; Assembly (none) -> FIT; MPN (none) -> CC0603KRX7R8BB105; Manufacturer (none) -> Yageo; Voltage (none) -> 25V
- C16: footprint Capacitor_SMD:C_0805_2012Metric -> ENKU:C_CC0805_YAGEO_REFLOW_TRANSFER; Assembly (none) -> FIT; MPN (none) -> CC0805KKX5R6BB106; Manufacturer (none) -> Yageo; Voltage (none) -> 10V
- C39: footprint Capacitor_SMD:C_0603_1608Metric -> ENKU:C_CC0603_YAGEO_REFLOW_TRANSFER; Assembly (none) -> FIT; MPN (none) -> CC0603JRNPO9BN102; Manufacturer (none) -> Yageo; Voltage (none) -> 50V
- R70: footprint Resistor_SMD:R_0603_1608Metric -> ENKU:R_RT0603_YAGEO_REFLOW; Assembly (none) -> FIT; MPN (none) -> RT0603BRD0726K7L; Manufacturer (none) -> Yageo
- R71: footprint Resistor_SMD:R_0603_1608Metric -> ENKU:R_RT0603_YAGEO_REFLOW; Assembly (none) -> FIT; MPN (none) -> RT0603BRD0710KL; Manufacturer (none) -> Yageo

Commit message: R128: reproduce ESP32-S3 module EP grid and audit actual mask/paste plots
U1 now uses nine nominal 0.9mm GND squares with explicit 0.8mm top-mask and paste apertures. Preserve twelve existing 0.3mm thermal drills/0.6mm lands; request both-side mask tents without claiming sealed, filled or qualified vias. Retain every old pad UUID/net/drill, all2639 copper items, placements, source nets, rules, outline/zones/RF restrictions and previous library bytes.

Add independent U1/reserved Octal-PSRAM/ambient guards, actual native mask/paste plot checks and intrinsic TL3340/USB hole audits. Keep all79 R127 exact part selections and numeric power checks. KiCad10.0.7 full local result: opens0/ERC0/parity0/DRC46(26library+20holes),425pads/117footprints. All12 independent guards and exact checkpoint comparison pass. Actual source-bound CI requested by workflow change; server_verified remains false until evidence captured.

Engineering source only. Active hole rule0.25mm and all20 findings retained. Mask/stencil/reflow, controlled SW1/FPC/stackup, bench and assembly acceptance remain open; fabrication_ready=false.
Parts:
- U1: footprint RF_Module:ESP32-S3-WROOM-1 -> ENKU:ESP32_S3_WROOM_1_N16R8_EP_GRID_03_TENT_REQUEST; EP Process (none) -> 9x0.9mm GND lands;9x0.8mm mask/paste;12x0.3mm PTH both-side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; MPN (none) -> ESP32-S3-WROOM-1-N16R8; Manufacturer (none) -> Espressif; Module Ambient (none) -> -40..65C by default;85C requires qualified PSRAM ECC firmwa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
Changed lines of the file:
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@@
 		(property "Reference" "U1" (at 63.55 65.55 0) (effects (font (size 0.88 0.88))))
 		(property "Value" "ESP32-S3-WROOM-1-N16R8" (at 101.55 65.55 0) (effects (font (size 0.88 0.88))))
-		(property "Footprint" "RF_Module:ESP32-S3-WROOM-1" (at 82.55 82.55 0) (effects (font (size 0.88 0.88)) (hide yes)))
+		(property "Footprint" "ENKU:ESP32_S3_WROOM_1_N16R8_EP_GRID_03_TENT_REQUEST" (at 82.55 82.55 0) (effects (font (size 0.88 0.88)) (hide yes)))
 		(property "Datasheet" "~" (at 82.55 82.55 0) (effects (font (size 0.88 0.88)) (hide yes)))
 		(property "Description" "ESP32-S3-WROOM-1-N16R8" (at 82.55 82.55 0) (effects (font (size 0.88 0.88)) (hide yes)))
@@
 		(pin "41")
 		(instances (project "enku-mainboard-r0.1" (path "/10000000-0000-4000-8000-000000000001/74000000-0000-4000-8000-000000000001" (reference "U1") (unit 1))))
+		(property "Manufacturer" "Espressif" (at 0 0 0) (effects (font (size .8 .8)) (hide yes)))
+		(property "MPN" "ESP32-S3-WROOM-1-N16R8" (at 0 0 0) (effects (font (size .8 .8)) (hide yes)))
+		(property "EP Process" "9x0.9mm GND lands;9x0.8mm mask/paste;12x0.3mm PTH both-side tent request;assembly acceptance pending" (at 0 0 0) (effects (font (size .8 .8)) (hide yes)))
+		(property "Module Ambient" "-40..65C by default;85C requires qualified PSRAM ECC firmware and1/16 capacity reduction" (at 0 0 0) (effects (font (size .8 .8)) (hide yes)))
 	)
 	(global_label "GND" (shape input) (at 60.96 58.42 0) (effects (font (size 0.88 0.88)) (justify right bottom)))
