File: hardware/mainboard/kicad/epd_hv.kicad_sch (KiCad schematic)
At the start: 33 parts, among them J3 FH34SRJ-24S-0.5SH(50), Q1 IRLML6346TRPBF

Commit message: hardware: preserve recovered R119 layout and verified R118 source [skip ci]
Persist the KiCad 10.0.7 project before the next routing pass. The recovered layout has 67 opens, ERC 0, parity 0 and zero RF keepout violations; routing is incomplete and fabrication is blocked. Preserve all pad and surviving copper net identities and retain an immutable R118 source archive.
Parts:
- L2: value 10uH TYS5040100M-10 -> 47uH TYS5040470M-10
Other:
- note added: "R118 requires first-board scope validation of VGH/VGL/VSH/VSL/VCOM. 47uH is the documented panel reference; 10uH is not an approved default. Pin 5 remains on hold pending vendor clarification."
- note added: "SSD1677 application circuit captured as discretes. R118 follows GDEY0397T81P supplied datasheet p19: 47uH + NMOS + 3x MBR0530 + 2.2R RESE + 1M GDR pulldown + local 4.7uF input capacitor."
- note removed: "R0.1 requires first-board scope validation of VGH/VGL/VSH/VSL/VCOM. TYS5040100M-10 and TYS5040470M-10 share the same TYS5040 land pattern, so 47uH remains a laboratory alternate without PCB respin."
- note removed: "SSD1677 application circuit captured as discretes. R0.1 now follows the current 3.97-inch panel reference: 10uH + NMOS + 3x MBR0530 + 2.2R RESE + 1M GDR pulldown + local 4.7uF input capacitor."
Changed lines of the file:
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@@
 	(symbol (lib_id "ENKU:L") (at 54.61 62.23 0) (unit 1) (exclude_from_sim no) (in_bom yes) (on_board yes) (dnp no)
 		(property "Reference" "L2" (at 49.61 48.23 0) (effects (font (size 0.9 0.9))))
-		(property "Value" "10uH TYS5040100M-10" (at 59.61 48.23 0) (effects (font (size 0.9 0.9))))
+		(property "Value" "47uH TYS5040470M-10" (at 59.61 48.23 0) (effects (font (size 0.9 0.9))))
 		(property "Footprint" "ENKU:TYS5040_5x5" (at 54.61 62.23 0) (effects (font (size 0.9 0.9)) (hide yes)))
 		(property "Datasheet" "~" (at 54.61 62.23 0) (effects (font (size 0.9 0.9)) (hide yes)))
-		(property "Description" "10uH TYS5040100M-10" (at 54.61 62.23 0) (effects (font (size 0.9 0.9)) (hide yes)))
+		(property "Description" "47uH TYS5040470M-10" (at 54.61 62.23 0) (effects (font (size 0.9 0.9)) (hide yes)))
 		(pin "1")
 		(pin "2")
@@
 	(global_label "GND" (shape input) (at 208.28 102.87 0) (effects (font (size 0.9 0.9)) (justify right bottom)))
 	(global_label "GND" (shape input) (at 247.65 102.87 180) (effects (font (size 0.9 0.9)) (justify right bottom)))
-	(text "SSD1677 application circuit captured as discretes. R0.1 now follows the current 3.97-inch panel reference: 10uH + NMOS + 3x MBR0530 + 2.2R RESE + 1M GDR pulldown + local 4.7uF input capacitor." (exclude_from_sim no) (at 25 20 0) (effects (font (size 1.0 1.0)) (justify left bottom)))
+	(text "SSD1677 application circuit captured as discretes. R118 follows GDEY0397T81P supplied datasheet p19: 47uH + NMOS + 3x MBR0530 + 2.2R RESE + 1M GDR pulldown + local 4.7uF input capacitor." (exclude_from_sim no) (at 25 20 0) (effects (font (size 1.0 1.0)) (justify left bottom)))
 	(text "D1: SW -> VGH. C3 flying capacitor + D2/D3 form the negative VGL pump. Q_EPD source is sensed at RESE through 2.2R to GND." (exclude_from_sim no) (at 25 25 0) (effects (font (size 1.0 1.0)) (justify left bottom)))
 	(text "VPP is explicitly left NC for normal operation; BS1 is tied LOW for 4-wire SPI. Current panel pins 6/7 remain NC pending panel-specific continuity confirmation." (exclude_from_sim no) (at 25 30 0) (effects (font (size 1.0 1.0)) (justify left bottom)))
-	(text "R0.1 requires first-board scope validation of VGH/VGL/VSH/VSL/VCOM. TYS5040100M-10 and TYS5040470M-10 share the same TYS5040 land pattern, so 47uH remains a laboratory alternate without PCB respin." (exclude_from_sim no) (at 25 35 0) (effects (font (size 1.0 1.0)) (justify left bottom)))
+	(text "R118 requires first-board scope validation of VGH/VGL/VSH/VSL/VCOM. 47uH is the documented panel reference; 10uH is not an approved default. Pin 5 remains on hold pending vendor clarification." (exclude_from_sim no) (at 25 35 0) (effects (font (size 1.0 1.0)) (justify left bottom)))
 	(symbol (lib_id "ENKU:TESTPOINT") (at 44.45 199.39 0) (unit 1) (exclude_from_sim no) (in_bom yes) (on_board yes) (dnp no)
 		(property "Reference" "TP9" (at 44.45 196.85 0) (effects (font (size 0.9 0.9))))

Commit message: R125: correct manufacturer Q1/Q2/U9 lands and guard full copper, netlist and assembly layers
Parts:
- Q1: footprint Package_TO_SOT_SMD:SOT-23 -> ENKU:IRLML6346_INFINEON_MICRO3
Changed lines of the file:
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@@
 		(property "Reference" "Q1" (at 77.455 68.55 0) (effects (font (size 0.9 0.9))))
 		(property "Value" "IRLML6346TRPBF" (at 91.455 68.55 0) (effects (font (size 0.9 0.9))))
-		(property "Footprint" "Package_TO_SOT_SMD:SOT-23" (at 84.455 82.55 0) (effects (font (size 0.9 0.9)) (hide yes)))
-		(property "Datasheet" "~" (at 84.455 82.55 0) (effects (font (size 0.9 0.9)) (hide yes)))
+		(property "Footprint" "ENKU:IRLML6346_INFINEON_MICRO3" (at 84.455 82.55 0) (effects (font (size 0.9 0.9)) (hide yes)))
+		(property "Datasheet" "https://www.infineon.com/assets/row/public/documents/24/49/infineon-irlml6346-datasheet-en.pdf" (at 84.455 82.55 0) (effects (font (size 0.9 0.9)) (hide yes)))
 		(property "Description" "IRLML6346TRPBF" (at 84.455 82.55 0) (effects (font (size 0.9 0.9)) (hide yes)))
 		(pin "1")

Commit message: R126: select 61 exact components, correct physical lands and local routing, preserve full source; NO FAB
Parts:
- C24, C25, C26, C31: footprint Capacitor_SMD:C_0805_2012Metric -> ENKU:C_CC0805_YAGEO_REFLOW_TRANSFER; Assembly (none) -> FIT; MPN (none) -> CC0805KKX7R8BB475; Manufacturer (none) -> Yageo; Voltage (none) -> 25V
- D1, D2, D3: value MBR0530 -> MBR0530T1G; footprint Diode_SMD:D_SOD-123 -> ENKU:MBR0530T1G_ONSEMI_CASE425H; Assembly (none) -> FIT; MPN (none) -> MBR0530T1G; Manufacturer (none) -> onsemi
- R28, R29: footprint Resistor_SMD:R_0603_1608Metric -> ENKU:R_RC0603_YAGEO_REFLOW; Assembly (none) -> FIT; MPN (none) -> RC0603JR-070RL; Manufacturer (none) -> Yageo
- R30, R31, R32, R33, R34: footprint Resistor_SMD:R_0603_1608Metric -> ENKU:R_RC0603_YAGEO_REFLOW; Assembly (none) -> FIT; MPN (none) -> RC0603FR-0722RL; Manufacturer (none) -> Yageo
- R35, R36: footprint Resistor_SMD:R_0603_1608Metric -> ENKU:R_RC0603_YAGEO_REFLOW; Assembly (none) -> FIT; MPN (none) -> RC0603FR-07100KL; Manufacturer (none) -> Yageo
- R38: footprint Resistor_SMD:R_0603_1608Metric -> ENKU:R_RC0603_YAGEO_REFLOW; Assembly (none) -> FIT; MPN (none) -> RC0603FR-071ML; Manufacturer (none) -> Yageo

Commit message: R127: finish passive MPN selection and correct USB VBUS capacitance
Select exact parts and nominal lands for the remaining 15 capacitors and R70/R71/R37. Reduce C4 from10uF/10V to1uF/25V, taking direct VBUS capacitance from15.8 to6.8uF. Preserve all417 original pad and2639 Cu identities/nets, with only3 declared EPD_VCI vertex adjustments.

Native KiCad10.0.7: opens0/ERC0/parity0/DRC47(27library+20holes). Add independent79-part, source and native-netlist numeric power guards. Record unqualified Ceff, inrush, EPD pulse/process gates; NO FAB.
Parts:
- C22, C23: footprint Capacitor_SMD:C_0603_1608Metric -> ENKU:C_CC0603_YAGEO_REFLOW_TRANSFER; Assembly (none) -> FIT; MPN (none) -> CC0603KRX7R8BB105; Manufacturer (none) -> Yageo; Voltage (none) -> 25V
- C27, C28, C29: footprint Capacitor_SMD:C_0805_2012Metric -> ENKU:C_CC0805_YAGEO_REFLOW_TRANSFER; Assembly (none) -> FIT; MPN (none) -> CC0805KKX7R8BB475; Manufacturer (none) -> Yageo; Voltage (none) -> 25V
- C30: footprint Capacitor_SMD:C_0805_2012Metric -> ENKU:C_CC0805_YAGEO_REFLOW_TRANSFER; Assembly (none) -> FIT; MPN (none) -> CC0805KKX7R8BB105; Manufacturer (none) -> Yageo; Voltage (none) -> 25V
- R37: footprint Resistor_SMD:R_0805_2012Metric -> ENKU:R_CRCW0805_HP_VISHAY_REFLOW; Assembly (none) -> FIT; MPN (none) -> CRCW08052R20FKEAHP; Manufacturer (none) -> Vishay
Changed lines of the file:
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@@
 		(property "Reference" "C22" (at 185.5 49.5 0) (effects (font (size 0.9 0.9))))
 		(property "Value" "1uF 25V" (at 195.5 49.5 0) (effects (font (size 0.9 0.9))))
-		(property "Footprint" "Capacitor_SMD:C_0603_1608Metric" (at 190.5 63.5 0) (effects (font (size 0.9 0.9)) (hide yes)))
-		(property "Datasheet" "~" (at 190.5 63.5 0) (effects (font (size 0.9 0.9)) (hide yes)))
+		(property "Footprint" "ENKU:C_CC0603_YAGEO_REFLOW_TRANSFER" (at 190.5 63.5 0) (effects (font (size 0.9 0.9)) (hide yes)))
+		(property "Datasheet" "https://yageogroup.com/download/specsheet/CC0603KRX7R8BB105" (at 190.5 63.5 0) (effects (font (size 0.9 0.9)) (hide yes)))
 		(property "Description" "1uF 25V" (at 190.5 63.5 0) (effects (font (size 0.9 0.9)) (hide yes)))
 		(pin "1")
 		(pin "2")
 		(instances (project "enku-mainboard-r0.1" (path "/10000000-0000-4000-8000-000000000001/72000000-0000-4000-8000-000000000055" (reference "C22") (unit 1))))
+		(property "MPN" "CC0603KRX7R8BB105" (at 0 0 0) (effects (font (size .8 .8)) (hide yes)))
+		(property "Manufacturer" "Yageo" (at 0 0 0) (effects (font (size .8 .8)) (hide yes)))
+		(property "Assembly" "FIT" (at 0 0 0) (effects (font (size .8 .8)) (hide yes)))
+		(property "Voltage" "25V" (at 0 0 0) (effects (font (size .8 .8)) (hide yes)))
 	)
 	(global_label "EPD_VCI" (shape input) (at 182.88 63.5 0) (effects (font (size 0.9 0.9)) (justify right bottom)))
@@
 		(property "Reference" "C23" (at 185.5 67.28 0) (effects (font (size 0.9 0.9))))
 		(property "Value" "1uF 25V" (at 195.5 67.28 0) (effects (font (size 0.9 0.9))))
-		(property "Footprint" "Capacitor_SMD:C_0603_1608Metric" (at 190.5 81.28 0) (effects (font (size 0.9 0.9)) (hide yes)))
-		(property "Datasheet" "~" (at 190.5 81.28 0) (effects (font (size 0.9 0.9)) (hide yes)))
+		(property "Footprint" "ENKU:C_CC0603_YAGEO_REFLOW_TRANSFER" (at 190.5 81.28 0) (effects (font (size 0.9 0.9)) (hide yes)))
+		(property "Datasheet" "https://yageogroup.com/download/specsheet/CC0603KRX7R8BB105" (at 190.5 81.28 0) (effects (font (size 0.9 0.9)) (hide yes)))
 		(property "Description" "1uF 25V" (at 190.5 81.28 0) (effects (font (size 0.9 0.9)) (hide yes)))
 		(pin "1")
 		(pin "2")
 		(instances (project "enku-mainboard-r0.1" (path "/10000000-0000-4000-8000-000000000001/72000000-0000-4000-8000-000000000060" (reference "C23") (unit 1))))
+		(property "MPN" "CC0603KRX7R8BB105" (at 0 0 0) (effects (font (size .8 .8)) (hide yes)))
+		(property "Manufacturer" "Yageo" (at 0 0 0) (effects (font (size .8 .8)) (hide yes)))
+		(property "Assembly" "FIT" (at 0 0 0) (effects (font (size .8 .8)) (hide yes)))
+		(property "Voltage" "25V" (at 0 0 0) (effects (font (size .8 .8)) (hide yes)))
 	)
 	(global_label "EPD_VDD" (shape input) (at 182.88 81.28 0) (effects (font (size 0.9 0.9)) (justify right bottom)))
@@
 		(property "Reference" "R37" (at 80.09 93.95 0) (effects (font (size 0.9 0.9))))
 		(property "Value" "2.2R 1% 0805" (at 90.09 93.95 0) (effects (font (size 0.9 0.9))))
-		(property "Footprint" "Resistor_SMD:R_0805_2012Metric" (at 85.09 107.95 0) (effects (font (size 0.9 0.9)) (hide yes)))
-		(property "Datasheet" "~" (at 85.09 107.95 0) (effects (font (size 0.9 0.9)) (hide yes)))
+		(property "Footprint" "ENKU:R_CRCW0805_HP_VISHAY_REFLOW" (at 85.09 107.95 0) (effects (font (size 0.9 0.9)) (hide yes)))
+		(property "Datasheet" "https://www.vishay.com/docs/20043/crcwhpe3.pdf" (at 85.09 107.95 0) (effects (font (size 0.9 0.9)) (hide yes)))
 		(property "Description" "2.2R 1% 0805" (at 85.09 107.95 0) (effects (font (size 0.9 0.9)) (hide yes)))
 		(pin "1")
 		(pin "2")
 		(instances (project "enku-mainboard-r0.1" (path "/10000000-0000-4000-8000-000000000001/72000000-0000-4000-8000-000000000117" (reference "R37") (unit 1))))
+		(property "MPN" "CRCW08052R20FKEAHP" (at 0 0 0) (effects (font (size .8 .8)) (hide yes)))
+		(property "Manufacturer" "Vishay" (at 0 0 0) (effects (font (size .8 .8)) (hide yes)))
+		(property "Assembly" "FIT" (at 0 0 0) (effects (font (size .8 .8)) (hide yes)))
 	)
 	(global_label "EPD_RESE" (shape input) (at 77.47 107.95 0) (effects (font (size 0.9 0.9)) (justify right bottom)))
@@
 		(property "Reference" "C27" (at 30.56 130.78 0) (effects (font (size 0.9 0.9))))
 		(property "Value" "4.7uF 25V" (at 40.56 130.78 0) (effects (font (size 0.9 0.9))))
-		(property "Footprint" "Capacitor_SMD:C_0805_2012Metric" (at 35.56 144.78 0) (effects (font (size 0.9 0.9)) (hide yes)))
-		(property "Datasheet" "~" (at 35.56 144.78 0) (effects (font (size 0.9 0.9)) (hide yes)))
+		(property "Footprint" "ENKU:C_CC0805_YAGEO_REFLOW_TRANSFER" (at 35.56 144.78 0) (effects (font (size 0.9 0.9)) (hide yes)))
+		(property "Datasheet" "https://yageogroup.com/download/specsheet/CC0805KKX7R8BB475" (at 35.56 144.78 0) (effects (font (size 0.9 0.9)) (hide yes)))
 		(property "Description" "4.7uF 25V" (at 35.56 144.78 0) (effects (font (size 0.9 0.9)) (hide yes)))
 		(pin "1")
 		(pin "2")
 		(instances (project "enku-mainboard-r0.1" (path "/10000000-0000-4000-8000-000000000001/72000000-0000-4000-8000-000000000152" (reference "C27") (unit 1))))
+		(property "MPN" "CC0805KKX7R8BB475" (at 0 0 0) (effects (font (size .8 .8)) (hide yes)))
+		(property "Manufacturer" "Yageo" (at 0 0 0) (effects (font (size .8 .8)) (hide yes)))
+		(property "Assembly" "FIT" (at 0 0 0) (effects (font (size .8 .8)) (hide yes)))
+		(property "Voltage" "25V" (at 0 0 0) (effects (font (size .8 .8)) (hide yes)))
 	)
 	(global_label "EPD_VSH1" (shape input) (at 27.94 144.78 0) (effects (font (size 0.9 0.9)) (justify right bottom)))
@@
 		(property "Reference" "C28" (at 59.77 130.78 0) (effects (font (size 0.9 0.9))))
 		(property "Value" "4.7uF 25V" (at 69.77 130.78 0) (effects (font (size 0.9 0.9))))
-		(property "Footprint" "Capacitor_SMD:C_0805_2012Metric" (at 64.77 144.78 0) (effects (font (size 0.9 0.9)) (hide yes)))
-		(property "Datasheet" "~" (at 64.77 144.78 0) (effects (font (size 0.9 0.9)) (hide yes)))
+		(property "Footprint" "ENKU:C_CC0805_YAGEO_REFLOW_TRANSFER" (at 64.77 144.78 0) (effects (font (size 0.9 0.9)) (hide yes)))
+		(property "Datasheet" "https://yageogroup.com/download/specsheet/CC0805KKX7R8BB475" (at 64.77 144.78 0) (effects (font (size 0.9 0.9)) (hide yes)))
 		(property "Description" "4.7uF 25V" (at 64.77 144.78 0) (effects (font (size 0.9 0.9)) (hide yes)))
 		(pin "1")
 		(pin "2")
 		(instances (project "enku-mainboard-r0.1" (path "/10000000-0000-4000-8000-000000000001/72000000-0000-4000-8000-000000000157" (reference "C28") (unit 1))))
+		(property "MPN" "CC0805KKX7R8BB475" (at 0 0 0) (effects (font (size .8 .8)) (hide yes)))
+		(property "Manufacturer" "Yageo" (at 0 0 0) (effects (font (size .8 .8)) (hide yes)))
+		(property "Assembly" "FIT" (at 0 0 0) (effects (font (size .8 .8)) (hide yes)))
+		(property "Voltage" "25V" (at 0 0 0) (effects (font (size .8 .8)) (hide yes)))
 	)
 	(global_label "EPD_VSH2" (shape input) (at 57.15 144.78 0) (effects (font (size 0.9 0.9)) (justify right bottom)))
@@
 		(property "Reference" "C29" (at 90.25 130.78 0) (effects (font (size 0.9 0.9))))
 		(property "Value" "4.7uF 25V" (at 100.25 130.78 0) (effects (font (size 0.9 0.9))))
-		(property "Footprint" "Capacitor_SMD:C_0805_2012Metric" (at 95.25 144.78 0) (effects (font (size 0.9 0.9)) (hide yes)))
-		(property "Datasheet" "~" (at 95.25 144.78 0) (effects (font (size 0.9 0.9)) (hide yes)))
+		(property "Footprint" "ENKU:C_CC0805_YAGEO_REFLOW_TRANSFER" (at 95.25 144.78 0) (effects (font (size 0.9 0.9)) (hide yes)))
+		(property "Datasheet" "https://yageogroup.com/download/specsheet/CC0805KKX7R8BB475" (at 95.25 144.78 0) (effects (font (size 0.9 0.9)) (hide yes)))
 		(property "Description" "4.7uF 25V" (at 95.25 144.78 0) (effects (font (size 0.9 0.9)) (hide yes)))
 		(pin "1")
 		(pin "2")
 		(instances (project "enku-mainboard-r0.1" (path "/10000000-0000-4000-8000-000000000001/72000000-0000-4000-8000-000000000162" (reference "C29") (unit 1))))
+		(property "MPN" "CC0805KKX7R8BB475" (at 0 0 0) (effects (font (size .8 .8)) (hide yes)))
+		(property "Manufacturer" "Yageo" (at 0 0 0) (effects (font (size .8 .8)) (hide yes)))
+		(property "Assembly" "FIT" (at 0 0 0) (effects (font (size .8 .8)) (hide yes)))
+		(property "Voltage" "25V" (at 0 0 0) (effects (font (size .8 .8)) (hide yes)))
 	)
 	(global_label "EPD_VSL" (shape input) (at 87.63 144.78 0) (effects (font (size 0.9 0.9)) (justify right bottom)))
@@
 		(property "Reference" "C30" (at 119.46 130.78 0) (effects (font (size 0.9 0.9))))
 		(property "Value" "1uF 25V X7R" (at 129.46 130.78 0) (effects (font (size 0.9 0.9))))
-		(property "Footprint" "Capacitor_SMD:C_0805_2012Metric" (at 124.46 144.78 0) (effects (font (size 0.9 0.9)) (hide yes)))
-		(property "Datasheet" "~" (at 124.46 144.78 0) (effects (font (size 0.9 0.9)) (hide yes)))
+		(property "Footprint" "ENKU:C_CC0805_YAGEO_REFLOW_TRANSFER" (at 124.46 144.78 0) (effects (font (size 0.9 0.9)) (hide yes)))
+		(property "Datasheet" "https://yageogroup.com/download/specsheet/CC0805KKX7R8BB105" (at 124.46 144.78 0) (effects (font (size 0.9 0.9)) (hide yes)))
 		(property "Description" "1uF 25V X7R" (at 124.46 144.78 0) (effects (font (size 0.9 0.9)) (hide yes)))
 		(pin "1")
 		(pin "2")
 		(instances (project "enku-mainboard-r0.1" (path "/10000000-0000-4000-8000-000000000001/72000000-0000-4000-8000-000000000167" (reference "C30") (unit 1))))
+		(property "MPN" "CC0805KKX7R8BB105" (at 0 0 0) (effects (font (size .8 .8)) (hide yes)))
+		(property "Manufacturer" "Yageo" (at 0 0 0) (effects (font (size .8 .8)) (hide yes)))
+		(property "Assembly" "FIT" (at 0 0 0) (effects (font (size .8 .8)) (hide yes)))
+		(property "Voltage" "25V" (at 0 0 0) (effects (font (size .8 .8)) (hide yes)))
 	)
 	(global_label "EPD_VCOM" (shape input) (at 116.84 144.78 0) (effects (font (size 0.9 0.9)) (justify right bottom)))
