File: hardware/mainboard/kicad/epd_hv.kicad_sch (KiCad schematic)
At the start: 33 parts, among them J3 FH34SRJ-24S-0.5SH(50), Q1 IRLML6346TRPBF

Commit message: R129: fix IC stencil apertures, pin-1 marking and native assembly classification
Verify six active IC pin maps and 97 native CPL placements. Preserve all 425 original pads, nets and 2639 tracks/vias; retain the 20 active intrinsic hole-clearance findings as fabrication gates. Add independent native KiCad checks and exact source-preservation guards.
Parts:
- J3: Assembly (none) -> FIT; MPN (none) -> FH34SRJ-24S-0.5SH(50); Manufacturer (none) -> Hirose
- TP10: footprint TestPoint:TestPoint_Pad_D1.5mm -> ENKU:SERVICE_PAD_D1_5_NO_PASTE; Assembly (none) -> BARE_PCB; Probe Label (none) -> RESE; now left out of the parts list
- TP11: footprint TestPoint:TestPoint_Pad_D1.5mm -> ENKU:SERVICE_PAD_D1_5_NO_PASTE; Assembly (none) -> BARE_PCB; Probe Label (none) -> VGH; now left out of the parts list
- TP12: footprint TestPoint:TestPoint_Pad_D1.5mm -> ENKU:SERVICE_PAD_D1_5_NO_PASTE; Assembly (none) -> BARE_PCB; Probe Label (none) -> VGL; now left out of the parts list
- TP13: footprint TestPoint:TestPoint_Pad_D1.5mm -> ENKU:SERVICE_PAD_D1_5_NO_PASTE; Assembly (none) -> BARE_PCB; Probe Label (none) -> VCOM; now left out of the parts list
- TP14: footprint TestPoint:TestPoint_Pad_D1.5mm -> ENKU:SERVICE_PAD_D1_5_NO_PASTE; Assembly (none) -> BARE_PCB; Probe Label (none) -> GND; now left out of the parts list
- TP9: footprint TestPoint:TestPoint_Pad_D1.5mm -> ENKU:SERVICE_PAD_D1_5_NO_PASTE; Assembly (none) -> BARE_PCB; Probe Label (none) -> GDR; now left out of the parts list
Changed lines of the file:
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@@
 		(property "Value" "FH34SRJ-24S-0.5SH(50)" (at 244.965 72.36 0) (effects (font (size 0.9 0.9))))
 		(property "Footprint" "ENKU:FH34SRJ-24S-0.5SH" (at 227.965 86.36 0) (effects (font (size 0.9 0.9)) (hide yes)))
-		(property "Datasheet" "~" (at 227.965 86.36 0) (effects (font (size 0.9 0.9)) (hide yes)))
+		(property "Datasheet" "https://www.hirose.com/product/en/products/FH34/FH34SRJ-24S-0.5SH%2850%29/" (at 227.965 86.36 0) (effects (font (size 0.9 0.9)) (hide yes)))
 		(property "Description" "FH34SRJ-24S-0.5SH(50)" (at 227.965 86.36 0) (effects (font (size 0.9 0.9)) (hide yes)))
 		(pin "1")
@@
 		(pin "S2")
 		(instances (project "enku-mainboard-r0.1" (path "/10000000-0000-4000-8000-000000000001/72000000-0000-4000-8000-000000000001" (reference "J3") (unit 1))))
+		(property "Manufacturer" "Hirose" (at 0 0 0) (effects (font (size .8 .8)) (hide yes)))
+		(property "MPN" "FH34SRJ-24S-0.5SH(50)" (at 0 0 0) (effects (font (size .8 .8)) (hide yes)))
+		(property "Assembly" "FIT" (at 0 0 0) (effects (font (size .8 .8)) (hide yes)))
 	)
 	(global_label "EPD_GDR" (shape input) (at 208.28 74.93 0) (effects (font (size 0.9 0.9)) (justify right bottom)))
@@
 	(text "VPP is explicitly left NC for normal operation; BS1 is tied LOW for 4-wire SPI. Current panel pins 6/7 remain NC pending panel-specific continuity confirmation." (exclude_from_sim no) (at 25 30 0) (effects (font (size 1.0 1.0)) (justify left bottom)))
 	(text "R118 requires first-board scope validation of VGH/VGL/VSH/VSL/VCOM. 47uH is the documented panel reference; 10uH is not an approved default. Pin 5 remains on hold pending vendor clarification." (exclude_from_sim no) (at 25 35 0) (effects (font (size 1.0 1.0)) (justify left bottom)))
-	(symbol (lib_id "ENKU:TESTPOINT") (at 44.45 199.39 0) (unit 1) (exclude_from_sim no) (in_bom yes) (on_board yes) (dnp no)
+	(symbol (lib_id "ENKU:TESTPOINT") (at 44.45 199.39 0) (unit 1) (exclude_from_sim no) (in_bom no) (on_board yes) (dnp no)
 		(property "Reference" "TP9" (at 44.45 196.85 0) (effects (font (size 0.9 0.9))))
 		(property "Value" "EPD_GDR" (at 44.45 201.93 0) (effects (font (size 0.9 0.9))))
-		(property "Footprint" "TestPoint:TestPoint_Pad_D1.5mm" (at 44.45 199.39 0) (effects (font (size 0.9 0.9)) (hide yes)))
+		(property "Footprint" "ENKU:SERVICE_PAD_D1_5_NO_PASTE" (at 44.45 199.39 0) (effects (font (size 0.9 0.9)) (hide yes)))
 		(property "Datasheet" "~" (at 44.45 199.39 0) (effects (font (size 0.9 0.9)) (hide yes)))
 		(property "Description" "ENKU R0.1 bring-up test point" (at 44.45 199.39 0) (effects (font (size 0.9 0.9)) (hide yes)))
 		(pin "1")
 		(instances (project "enku-mainboard-r0.1" (path "/10000000-0000-4000-8000-000000000001/75100000-0000-4000-8000-000000000001" (reference "TP9") (unit 1))))
+		(property "Assembly" "BARE_PCB" (at 0 0 0) (effects (font (size .8 .8)) (hide yes)))
+		(property "Probe Label" "GDR" (at 0 0 0) (effects (font (size .8 .8)) (hide yes)))
 	)
 	(global_label "EPD_GDR" (shape bidirectional) (at 40.64 199.39 0)
 		(effects (font (size 0.9 0.9)) (justify right bottom))
 )
-	(symbol (lib_id "ENKU:TESTPOINT") (at 80.01 199.39 0) (unit 1) (exclude_from_sim no) (in_bom yes) (on_board yes) (dnp no)
+	(symbol (lib_id "ENKU:TESTPOINT") (at 80.01 199.39 0) (unit 1) (exclude_from_sim no) (in_bom no) (on_board yes) (dnp no)
 		(property "Reference" "TP10" (at 80.01 196.85 0) (effects (font (size 0.9 0.9))))
 		(property "Value" "EPD_RESE" (at 80.01 201.93 0) (effects (font (size 0.9 0.9))))
-		(property "Footprint" "TestPoint:TestPoint_Pad_D1.5mm" (at 80.01 199.39 0) (effects (font (size 0.9 0.9)) (hide yes)))
+		(property "Footprint" "ENKU:SERVICE_PAD_D1_5_NO_PASTE" (at 80.01 199.39 0) (effects (font (size 0.9 0.9)) (hide yes)))
 		(property "Datasheet" "~" (at 80.01 199.39 0) (effects (font (size 0.9 0.9)) (hide yes)))
 		(property "Description" "ENKU R0.1 bring-up test point" (at 80.01 199.39 0) (effects (font (size 0.9 0.9)) (hide yes)))
 		(pin "1")
 		(instances (project "enku-mainboard-r0.1" (path "/10000000-0000-4000-8000-000000000001/75100000-0000-4000-8000-000000000004" (reference "TP10") (unit 1))))
+		(property "Assembly" "BARE_PCB" (at 0 0 0) (effects (font (size .8 .8)) (hide yes)))
+		(property "Probe Label" "RESE" (at 0 0 0) (effects (font (size .8 .8)) (hide yes)))
 	)
 	(global_label "EPD_RESE" (shape bidirectional) (at 76.2 199.39 0)
 		(effects (font (size 0.9 0.9)) (justify right bottom))
 )
-	(symbol (lib_id "ENKU:TESTPOINT") (at 115.57 199.39 0) (unit 1) (exclude_from_sim no) (in_bom yes) (on_board yes) (dnp no)
+	(symbol (lib_id "ENKU:TESTPOINT") (at 115.57 199.39 0) (unit 1) (exclude_from_sim no) (in_bom no) (on_board yes) (dnp no)
 		(property "Reference" "TP11" (at 115.57 196.85 0) (effects (font (size 0.9 0.9))))
 		(property "Value" "EPD_VGH" (at 115.57 201.93 0) (effects (font (size 0.9 0.9))))
-		(property "Footprint" "TestPoint:TestPoint_Pad_D1.5mm" (at 115.57 199.39 0) (effects (font (size 0.9 0.9)) (hide yes)))
+		(property "Footprint" "ENKU:SERVICE_PAD_D1_5_NO_PASTE" (at 115.57 199.39 0) (effects (font (size 0.9 0.9)) (hide yes)))
 		(property "Datasheet" "~" (at 115.57 199.39 0) (effects (font (size 0.9 0.9)) (hide yes)))
 		(property "Description" "ENKU R0.1 bring-up test point" (at 115.57 199.39 0) (effects (font (size 0.9 0.9)) (hide yes)))
 		(pin "1")
 		(instances (project "enku-mainboard-r0.1" (path "/10000000-0000-4000-8000-000000000001/75100000-0000-4000-8000-000000000007" (reference "TP11") (unit 1))))
+		(property "Assembly" "BARE_PCB" (at 0 0 0) (effects (font (size .8 .8)) (hide yes)))
+		(property "Probe Label" "VGH" (at 0 0 0) (effects (font (size .8 .8)) (hide yes)))
 	)
 	(global_label "EPD_VGH" (shape bidirectional) (at 111.76 199.39 0)
 		(effects (font (size 0.9 0.9)) (justify right bottom))
 )
-	(symbol (lib_id "ENKU:TESTPOINT") (at 149.86 199.39 0) (unit 1) (exclude_from_sim no) (in_bom yes) (on_board yes) (dnp no)
+	(symbol (lib_id "ENKU:TESTPOINT") (at 149.86 199.39 0) (unit 1) (exclude_from_sim no) (in_bom no) (on_board yes) (dnp no)
 		(property "Reference" "TP12" (at 149.86 196.85 0) (effects (font (size 0.9 0.9))))
 		(property "Value" "EPD_VGL" (at 149.86 201.93 0) (effects (font (size 0.9 0.9))))
-		(property "Footprint" "TestPoint:TestPoint_Pad_D1.5mm" (at 149.86 199.39 0) (effects (font (size 0.9 0.9)) (hide yes)))
+		(property "Footprint" "ENKU:SERVICE_PAD_D1_5_NO_PASTE" (at 149.86 199.39 0) (effects (font (size 0.9 0.9)) (hide yes)))
 		(property "Datasheet" "~" (at 149.86 199.39 0) (effects (font (size 0.9 0.9)) (hide yes)))
 		(property "Description" "ENKU R0.1 bring-up test point" (at 149.86 199.39 0) (effects (font (size 0.9 0.9)) (hide yes)))
 		(pin "1")
 		(instances (project "enku-mainboard-r0.1" (path "/10000000-0000-4000-8000-000000000001/75100000-0000-4000-8000-000000000010" (reference "TP12") (unit 1))))
+		(property "Assembly" "BARE_PCB" (at 0 0 0) (effects (font (size .8 .8)) (hide yes)))
+		(property "Probe Label" "VGL" (at 0 0 0) (effects (font (size .8 .8)) (hide yes)))
 	)
 	(global_label "EPD_VGL" (shape bidirectional) (at 146.05 199.39 0)
 		(effects (font (size 0.9 0.9)) (justify right bottom))
 )
-	(symbol (lib_id "ENKU:TESTPOINT") (at 185.42 199.39 0) (unit 1) (exclude_from_sim no) (in_bom yes) (on_board yes) (dnp no)
+	(symbol (lib_id "ENKU:TESTPOINT") (at 185.42 199.39 0) (unit 1) (exclude_from_sim no) (in_bom no) (on_board yes) (dnp no)
 		(property "Reference" "TP13" (at 185.42 196.85 0) (effects (font (size 0.9 0.9))))
 		(property "Value" "EPD_VCOM" (at 185.42 201.93 0) (effects (font (size 0.9 0.9))))
-		(property "Footprint" "TestPoint:TestPoint_Pad_D1.5mm" (at 185.42 199.39 0) (effects (font (size 0.9 0.9)) (hide yes)))
+		(property "Footprint" "ENKU:SERVICE_PAD_D1_5_NO_PASTE" (at 185.42 199.39 0) (effects (font (size 0.9 0.9)) (hide yes)))
 		(property "Datasheet" "~" (at 185.42 199.39 0) (effects (font (size 0.9 0.9)) (hide yes)))
 		(property "Description" "ENKU R0.1 bring-up test point" (at 185.42 199.39 0) (effects (font (size 0.9 0.9)) (hide yes)))
 		(pin "1")
 		(instances (project "enku-mainboard-r0.1" (path "/10000000-0000-4000-8000-000000000001/75100000-0000-4000-8000-000000000013" (reference "TP13") (unit 1))))
+		(property "Assembly" "BARE_PCB" (at 0 0 0) (effects (font (size .8 .8)) (hide yes)))
+		(property "Probe Label" "VCOM" (at 0 0 0) (effects (font (size .8 .8)) (hide yes)))
 	)
 	(global_label "EPD_VCOM" (shape bidirectional) (at 181.61 199.39 0)
 		(effects (font (size 0.9 0.9)) (justify right bottom))
 )
-	(symbol (lib_id "ENKU:TESTPOINT") (at 219.71 199.39 0) (unit 1) (exclude_from_sim no) (in_bom yes) (on_board yes) (dnp no)
+	(symbol (lib_id "ENKU:TESTPOINT") (at 219.71 199.39 0) (unit 1) (exclude_from_sim no) (in_bom no) (on_board yes) (dnp no)
 		(property "Reference" "TP14" (at 219.71 196.85 0) (effects (font (size 0.9 0.9))))
 		(property "Value" "GND" (at 219.71 201.93 0) (effects (font (size 0.9 0.9))))
-		(property "Footprint" "TestPoint:TestPoint_Pad_D1.5mm" (at 219.71 199.39 0) (effects (font (size 0.9 0.9)) (hide yes)))
+		(property "Footprint" "ENKU:SERVICE_PAD_D1_5_NO_PASTE" (at 219.71 199.39 0) (effects (font (size 0.9 0.9)) (hide yes)))
 		(property "Datasheet" "~" (at 219.71 199.39 0) (effects (font (size 0.9 0.9)) (hide yes)))
 		(property "Description" "ENKU R0.1 bring-up test point" (at 219.71 199.39 0) (effects (font (size 0.9 0.9)) (hide yes)))
 		(pin "1")
 		(instances (project "enku-mainboard-r0.1" (path "/10000000-0000-4000-8000-000000000001/75100000-0000-4000-8000-000000000016" (reference "TP14") (unit 1))))
+		(property "Assembly" "BARE_PCB" (at 0 0 0) (effects (font (size .8 .8)) (hide yes)))
+		(property "Probe Label" "GND" (at 0 0 0) (effects (font (size .8 .8)) (hide yes)))
 	)
 	(global_label "GND" (shape bidirectional) (at 215.9 199.39 0)

Commit message: R130 BAT-REV3: PH2 battery and separate NTC; correct Laird lands and preserve R129
Implement the two-wire battery interface, retain all accepted copper identities, and restore the L2 land/via correction. Add native source/assembly/plot guards, supplier evidence and dimensional studies. Charging temperature, capacity/timer, complete mechanical fit and twenty hole findings remain HOLD; no fabrication or orders.
Parts:
- L2: footprint ENKU:TYS5040_5x5 -> ENKU:TYS5040_LAIRD_G42_T14_H23; Assembly (none) -> FIT; MPN (none) -> TYS5040470M-10; Manufacturer (none) -> Laird Performance Materials
- Q1: Assembly (none) -> FIT; MPN (none) -> IRLML6346TRPBF; Manufacturer (none) -> Infineon
Changed lines of the file:
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@@
 		(property "Reference" "L2" (at 49.61 48.23 0) (effects (font (size 0.9 0.9))))
 		(property "Value" "47uH TYS5040470M-10" (at 59.61 48.23 0) (effects (font (size 0.9 0.9))))
-		(property "Footprint" "ENKU:TYS5040_5x5" (at 54.61 62.23 0) (effects (font (size 0.9 0.9)) (hide yes)))
-		(property "Datasheet" "~" (at 54.61 62.23 0) (effects (font (size 0.9 0.9)) (hide yes)))
+		(property "Footprint" "ENKU:TYS5040_LAIRD_G42_T14_H23" (at 54.61 62.23 0) (effects (font (size 0.9 0.9)) (hide yes)))
+		(property "Datasheet" "https://www.laird.com/sites/default/files/tys5040-series-datasheet.pdf" (at 54.61 62.23 0) (effects (font (size 0.9 0.9)) (hide yes)))
 		(property "Description" "47uH TYS5040470M-10" (at 54.61 62.23 0) (effects (font (size 0.9 0.9)) (hide yes)))
 		(pin "1")
 		(pin "2")
 		(instances (project "enku-mainboard-r0.1" (path "/10000000-0000-4000-8000-000000000001/72000000-0000-4000-8000-000000000105" (reference "L2") (unit 1))))
+		(property "Manufacturer" "Laird Performance Materials" (at 0 0 0) (effects (font (size .8 .8)) (hide yes)))
+		(property "MPN" "TYS5040470M-10" (at 0 0 0) (effects (font (size .8 .8)) (hide yes)))
+		(property "Assembly" "FIT" (at 0 0 0) (effects (font (size .8 .8)) (hide yes)))
 	)
 	(global_label "EPD_VCI" (shape input) (at 46.99 62.23 0) (effects (font (size 0.9 0.9)) (justify right bottom)))
@@
 		(pin "2")
 		(instances (project "enku-mainboard-r0.1" (path "/10000000-0000-4000-8000-000000000001/72000000-0000-4000-8000-000000000110" (reference "Q1") (unit 1))))
+		(property "Manufacturer" "Infineon" (at 0 0 0) (effects (font (size .8 .8)) (hide yes)))
+		(property "MPN" "IRLML6346TRPBF" (at 0 0 0) (effects (font (size .8 .8)) (hide yes)))
+		(property "Assembly" "FIT" (at 0 0 0) (effects (font (size .8 .8)) (hide yes)))
 	)
 	(global_label "EPD_GDR" (shape input) (at 74.93 81.28 0) (effects (font (size 0.9 0.9)) (justify right bottom)))
