File: hardware/mainboard/kicad/power.kicad_sch (KiCad schematic)
At the start: 33 parts, among them J1 1S LiPo + NTC, Q2 AO3401A, SW1 MK-12C03-G015, U3 BQ25185DLHR, U4 TPS63802DLAR

Commit message: R130 BAT-REV3: PH2 battery and separate NTC; correct Laird lands and preserve R129
Implement the two-wire battery interface, retain all accepted copper identities, and restore the L2 land/via correction. Add native source/assembly/plot guards, supplier evidence and dimensional studies. Charging temperature, capacity/timer, complete mechanical fit and twenty hole findings remain HOLD; no fabrication or orders.
Parts:
- added J8: External cell NTC / hand solder, ENKU:NTC_WIRE_TERMINALS_TS_BAR_GND_NO_PASTE, symbol ENKU:NTC_WIRE2
- J1: value 1S LiPo + NTC -> 1S LiPo PCM / PH-2; footprint ENKU:JST_PH_S3B-PH-SM4-TB_1x03-1MP_P2.00mm_Horizontal -> ENKU:JST_PH_S2B-PH-SM4-TB_1x02-1MP_P2.00mm_Horizontal; symbol ENKU:BAT3 -> ENKU:BAT2; Assembly (none) -> FIT; Battery Interface (none) -> PHR-2: cavity1 VBAT+, cavity2 GND; battery wire colors do n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; Crimp Contact (none) -> JST SPH-002T-P0.5S; AWG30-24, insulation0.8-1.5mm; tooling/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; MPN (none) -> S2B-PH-SM4-TB(LF)(SN); Manufacturer (none) -> JST; Mating Housing (none) -> JST PHR-2
- L1: Assembly (none) -> FIT; MPN (none) -> DFE201612E-R47M=P2; Manufacturer (none) -> Murata
- Q2: Assembly (none) -> FIT; MPN (none) -> AO3401A; Manufacturer (none) -> Alpha & Omega Semiconductor
- SW1: Assembly (none) -> FIT; MPN (none) -> MK-12C03-G015; Manufacturer (none) -> G-Switch
- U3: Battery Qualification (none) -> No battery/thermal/current/PCM approval; no manufacture; Charge Profile 4.2V/500mA input/300mA fast charge;RevB timer360min;battery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 -> HOLD BAT-REV3: 4.2V / 500mA IN / nominal300mA; RevB timer36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
Connections:
- net BAT_TS: now also J8.1 (TS/MR); no longer J1.3 (NTC)
- net GND: now also J8.2 (GND)
Other:
- note added: "BAT-REV3 HOLD: actual NTC retained on CELL. No fixed resistor. 3435K direct TS needs0-45C protection redesign. 300mA/6h timer not qualified for2-2.5Ah."
Changed lines of the file:
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@@
 		(property "MPN" "BQ25185DLHR" (at 0 0 0) (effects (font (size .8 .8)) (hide yes)))
 		(property "Assembly" "FIT" (at 0 0 0) (effects (font (size .8 .8)) (hide yes)))
-		(property "Charge Profile" "4.2V/500mA input/300mA fast charge;RevB timer360min;battery NTC and capacity qualification pending" (at 0 0 0) (effects (font (size .8 .8)) (hide yes)))
+		(property "Charge Profile" "HOLD BAT-REV3: 4.2V / 500mA IN / nominal300mA; RevB timer360min incompatible with assured full2500mAh recharge; direct3435K NTC hot threshold exceeds45C" (at 0 0 0) (effects (font (size .8 .8)) (hide yes)))
+		(property "Battery Qualification" "No battery/thermal/current/PCM approval; no manufacture" (at 0 0 0) (effects (font (size .8 .8)) (hide yes)))
 	)
 	(global_label "VSYS" (shape output) (at 148.59 55.88 180) (effects (font (size 0.95 0.95)) (justify right bottom)))
@@
 	(global_label "GND" (shape output) (at 220.98 63.5 180) (effects (font (size 0.95 0.95)) (justify right bottom)))
 	(global_label "REG_FB" (shape output) (at 220.98 60.96 180) (effects (font (size 0.95 0.95)) (justify right bottom)))
-	(symbol (lib_id "ENKU:BAT3") (at 135.255 125.73 0) (unit 1) (exclude_from_sim no) (in_bom yes) (on_board yes) (dnp no)
+	(symbol (lib_id "ENKU:BAT2") (at 135.255 125.73 0) (unit 1) (exclude_from_sim no) (in_bom yes) (on_board yes) (dnp no)
 		(property "Reference" "J1" (at 128.255 109.73 0) (effects (font (size 0.95 0.95))))
-		(property "Value" "1S LiPo + NTC" (at 142.255 109.73 0) (effects (font (size 0.95 0.95))))
-		(property "Footprint" "ENKU:JST_PH_S3B-PH-SM4-TB_1x03-1MP_P2.00mm_Horizontal" (at 135.255 125.73 0) (effects (font (size 0.95 0.95)) (hide yes)))
-		(property "Datasheet" "~" (at 135.255 125.73 0) (effects (font (size 0.95 0.95)) (hide yes)))
-		(property "Description" "1S LiPo + NTC" (at 135.255 125.73 0) (effects (font (size 0.95 0.95)) (hide yes)))
-		(pin "1")
-		(pin "2")
-		(pin "3")
+		(property "Value" "1S LiPo PCM / PH-2" (at 142.255 109.73 0) (effects (font (size 0.95 0.95))))
+		(property "Footprint" "ENKU:JST_PH_S2B-PH-SM4-TB_1x02-1MP_P2.00mm_Horizontal" (at 135.255 125.73 0) (effects (font (size 0.95 0.95)) (hide yes)))
+		(property "Datasheet" "https://www.jst-mfg.com/product/pdf/eng/ePH.pdf" (at 135.255 125.73 0) (effects (font (size 0.95 0.95)) (hide yes)))
+		(property "Description" "Protected standard TWO-wire LiPo; separate J8 cell-temperature sensor" (at 135.255 125.73 0) (effects (font (size 0.95 0.95)) (hide yes)))
+		(pin "1")
+		(pin "2")
 		(instances (project "enku-mainboard-r0.1" (path "/10000000-0000-4000-8000-000000000001/70000000-0000-4000-8000-000000000072" (reference "J1") (unit 1))))
+		(property "Battery Interface" "PHR-2: cavity1 VBAT+, cavity2 GND; battery wire colors do not prove polarity" (at 0 0 0) (effects (font (size .8 .8)) (hide yes)))
+		(property "Mating Housing" "JST PHR-2" (at 0 0 0) (effects (font (size .8 .8)) (hide yes)))
+		(property "Crimp Contact" "JST SPH-002T-P0.5S; AWG30-24, insulation0.8-1.5mm; tooling/pull test pending" (at 0 0 0) (effects (font (size .8 .8)) (hide yes)))
+		(property "Manufacturer" "JST" (at 0 0 0) (effects (font (size .8 .8)) (hide yes)))
+		(property "MPN" "S2B-PH-SM4-TB(LF)(SN)" (at 0 0 0) (effects (font (size .8 .8)) (hide yes)))
+		(property "Assembly" "FIT" (at 0 0 0) (effects (font (size .8 .8)) (hide yes)))
 	)
 	(global_label "VBAT" (shape input) (at 125.73 125.73 0) (effects (font (size 0.95 0.95)) (justify right bottom)))
 	(global_label "GND" (shape output) (at 144.78 124.46 180) (effects (font (size 0.95 0.95)) (justify right bottom)))
-	(global_label "BAT_TS" (shape output) (at 144.78 127 180) (effects (font (size 0.95 0.95)) (justify right bottom)))
 	(symbol (lib_id "ENKU:C") (at 27.94 82.55 0) (unit 1) (exclude_from_sim no) (in_bom yes) (on_board yes) (dnp no)
 		(property "Reference" "C2" (at 22.94 66.55 0) (effects (font (size 0.95 0.95))))
@@
 		(pin "3")
 		(instances (project "enku-mainboard-r0.1" (path "/10000000-0000-4000-8000-000000000001/70000000-0000-4000-8000-000000000179" (reference "SW1") (unit 1))))
+		(property "Manufacturer" "G-Switch" (at 0 0 0) (effects (font (size .8 .8)) (hide yes)))
+		(property "MPN" "MK-12C03-G015" (at 0 0 0) (effects (font (size .8 .8)) (hide yes)))
+		(property "Assembly" "FIT" (at 0 0 0) (effects (font (size .8 .8)) (hide yes)))
 	)
 	(global_label "PWR_GATE" (shape input) (at 196.85 127 0) (effects (font (size 0.95 0.95)) (justify right bottom)))
@@
 		(property "Value" "0.47uH DFE201612E-R47M=P2" (at 209.47 84.33 0) (effects (font (size 0.95 0.95))))
 		(property "Footprint" "ENKU:Murata_DFE201612E" (at 204.47 100.33 0) (effects (font (size 0.95 0.95)) (hide yes)))
-		(property "Datasheet" "~" (at 204.47 100.33 0) (effects (font (size 0.95 0.95)) (hide yes)))
+		(property "Datasheet" "https://pim.murata.com/asset/pim4/inductor/J%28E%29TE243A-0006_PDF_INDUCTOR" (at 204.47 100.33 0) (effects (font (size 0.95 0.95)) (hide yes)))
 		(property "Description" "Murata DFE201612E-R47M=P2, 0.47uH, 4.5A rated, 5.5A Isat" (at 204.47 100.33 0) (effects (font (size 0.95 0.95)) (hide yes)))
 		(pin "1")
 		(pin "2")
 		(instances (project "enku-mainboard-r0.1" (path "/10000000-0000-4000-8000-000000000001/70000000-0000-4000-8000-000000000189" (reference "L1") (unit 1))))
+		(property "Manufacturer" "Murata" (at 0 0 0) (effects (font (size .8 .8)) (hide yes)))
+		(property "MPN" "DFE201612E-R47M=P2" (at 0 0 0) (effects (font (size .8 .8)) (hide yes)))
+		(property "Assembly" "FIT" (at 0 0 0) (effects (font (size .8 .8)) (hide yes)))
 	)
 	(global_label "REG_L1" (shape input) (at 196.85 100.33 0) (effects (font (size 0.95 0.95)) (justify right bottom)))
@@
  (pin "2")
  (instances (project "enku-mainboard-r0.1" (path "/10000000-0000-4000-8000-000000000001/e5100000-0000-4000-8000-000000000001" (reference "Q2") (unit 1))))
-)
+		(property "Manufacturer" "Alpha & Omega Semiconductor" (at 0 0 0) (effects (font (size .8 .8)) (hide yes)))
+		(property "MPN" "AO3401A" (at 0 0 0) (effects (font (size .8 .8)) (hide yes)))
+		(property "Assembly" "FIT" (at 0 0 0) (effects (font (size .8 .8)) (hide yes)))
+	)
 	(symbol (lib_id "ENKU:R") (at 320.04 143.51 0) (unit 1) (exclude_from_sim no) (in_bom yes) (on_board yes) (dnp no)
  (property "Reference" "R40" (at 315.04 127.50999999999999 0) (effects (font (size 0.95 0.95))))
@@
 	(global_label "PWR_GATE" (shape output) (at 327.66 143.51 180) (effects (font (size 0.95 0.95)) (justify right bottom)))
 (no_connect (at 205.74 134.62))
-)
+(symbol (lib_id "ENKU:NTC_WIRE2") (at 135.255 148.59 0) (unit 1) (exclude_from_sim no) (in_bom no) (on_board yes) (dnp no)
+   (property "Reference" "J8" (at 135.255 143.59 0) (effects (font (size .95 .95))))
+   (property "Value" "External cell NTC / hand solder" (at 135.255 153.59 0) (effects (font (size .95 .95))))
+   (property "Footprint" "ENKU:NTC_WIRE_TERMINALS_TS_BAR_GND_NO_PASTE" (at 135.255 148.59 0) (effects (font (size .95 .95)) (hide yes)))
+   (pin "1")
+   (pin "2")
+   (instances (project "enku-mainboard-r0.1" (path "/10000000-0000-4000-8000-000000000001/daaa0800-0000-4000-8000-000000000008" (reference "J8") (unit 1))))
+		(property "Assembly" "BARE_PCB" (at 0 0 0) (effects (font (size .8 .8)) (hide yes)))
+		(property "Sensor MPN Candidate" "Semitec 103JT-050" (at 0 0 0) (effects (font (size .8 .8)) (hide yes)))
+		(property "Sensor Status" "10k +/-1%, B25/85 3435K +/-1%; direct TS hot limit is NOT qualified for0-45C pack" (at 0 0 0) (effects (font (size .8 .8)) (hide yes)))
+		(property "Assembly Process" "Hand solder insulated sensor tails; sensor film stays <150C; minimum7mm bend distance, separate strain relief required" (at 0 0 0) (effects (font (size .8 .8)) (hide yes)))
+		(property "Thermal Attachment" "Retained flat against replaceable pouch, insulation/no pressure; mechanical retention and replacement test pending" (at 0 0 0) (effects (font (size .8 .8)) (hide yes)))
+	)
+   (global_label "BAT_TS" (shape output) (at 125.73 148.59 0) (effects (font (size .95 .95)) (justify left bottom)))
+   (global_label "GND" (shape output) (at 144.78 148.59 180) (effects (font (size .95 .95)) (justify right bottom)))
+   (text "BAT-REV3 HOLD: actual NTC retained on CELL. No fixed resistor. 3435K direct TS needs0-45C protection redesign. 300mA/6h timer not qualified for2-2.5Ah." (at 185 170 0) (effects (font (size 1 1)) (justify left)))
+ )

Commit message: R132 recovery checkpoint: reconstruct voltage-TS power path; routing incomplete NO FAB
Parts:
- added R80: 31.6k 1%, ENKU:R_RC0603_YAGEO_REFLOW, symbol ENKU:R
- added R81: 19.6k 1%, ENKU:R_RC0603_YAGEO_REFLOW, symbol ENKU:R
- added R82: 100k 1%, ENKU:R_RC0603_YAGEO_REFLOW, symbol ENKU:R
- added R83: 69.8k 1%, ENKU:R_RC0603_YAGEO_REFLOW, symbol ENKU:R
- C7: value 10uF 25V -> 22uF 10V; MPN CC0805KKX5R8BB106 -> CC0805MKX5R6BB226; Voltage 25V -> 10V
- C8: value 4.7uF 10V -> 22uF 10V; MPN CC0805KKX5R6BB475 -> CC0805MKX5R6BB226
- J8: Sensor Status 10k +/-1%, B25/85 3435K +/-1%; direct TS hot limit is NOT q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 -> Real103JT-050; R132 voltage-TS model guards5-40C, absolute0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
- R12: value 10k DNP -> 10k; Assembly DNP -> FIT; now fitted
- R8: value 18k 1% -> 3.48k 1%; MPN RC0603FR-0718KL -> RC0603FR-073K48L
- R9: value 1k 1% -> 2k 1%; MPN RC0603FR-071KL -> RC0603FR-072KL
- U3: value BQ25185DLHR -> BQ24072TRGTR; footprint ENKU:BQ25185_DLH0010A_TI_STENCIL -> ENKU:BQ24072T_RGT0016C_TI; symbol ENKU:BQ25185_DLH -> ENKU:BQ24072T_RGT; Charge Profile HOLD BAT-REV3: 4.2V / 500mA IN / nominal300mA; RevB timer36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 -> R132 445mA nominal; USB500 max500mA; voltage-TS guarded win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; MPN BQ25185DLHR -> BQ24072TRGTR
Connections:
- net BAT_TS: now also R80.2, R81.1, R82.1; no longer U3.6 (TS/MR)
- net CHG_ILIM_VSET: now also U3.12 (ILIM); no longer U3.7 (ILIM/VSET)
- net CHG_ISET: now also U3.16 (ISET); no longer U3.8 (ISET)
- net CHG_STAT1: now also U3.7 (PGOOD_N); no longer U3.9 (STAT1)
- net CHG_STAT2: now also U3.9 (CHG_N); no longer U3.3 (STAT2)
- net GND: now also U3.15 (TD), U3.17 (EP), U3.8 (EN2), R81.2, R83.2; no longer U3.11 (EP)
- net VBAT: now also U3.3 (BAT)
- net VBUS_USB: now also U3.13 (IN), U3.6 (EN1), R80.1; no longer U3.10 (IN)
- net VSYS: now also U3.10 (OUT), U3.11 (OUT); no longer U3.1 (SYS)
- new net CHG_TMR: R83.1, U3.14 (TMR)
- new net CHG_TS: R82.2, U3.1 (TS)
Other:
- note added: "R132: real retained cell NTC. Nominal guarded5-40C window,445mA/8.725h; full-cycle and thermal hardware qualification HOLD."
- note removed: "BAT-REV3 HOLD: actual NTC retained on CELL. No fixed resistor. 3435K direct TS needs0-45C protection redesign. 300mA/6h timer not qualified for2-2.5Ah."
