File: hardware/mainboard/kicad/connectors.kicad_sch (KiCad schematic)
At the start: 10 parts, among them J5 GCT USB4105-GF-A-120, J7 Tag-Connect TC2030-IDC-NL, U8 USBLC6-2SC6

Commit message: R129: fix IC stencil apertures, pin-1 marking and native assembly classification
Verify six active IC pin maps and 97 native CPL placements. Preserve all 425 original pads, nets and 2639 tracks/vias; retain the 20 active intrinsic hole-clearance findings as fabrication gates. Add independent native KiCad checks and exact source-preservation guards.
Parts:
- J5: footprint Connector_USB:USB_C_Receptacle_GCT_USB4105-xx-A_16P_TopMnt_Horizontal -> ENKU:USB4105_EXISTING_LANDS_SHIELD_S
- J7: footprint Connector:Tag-Connect_TC2030-IDC-NL_2x03_P1.27mm_Vertical -> ENKU:TC2030_NL_CONTACTS_PIN1; Assembly (none) -> BARE_PCB
- U8: Assembly (none) -> FIT; MPN (none) -> USBLC6-2SC6; Manufacturer (none) -> STMicroelectronics
Changed lines of the file:
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@@
 		(property "Reference" "J5" (at 49.77 66.55 0) (effects (font (size 0.9 0.9))))
 		(property "Value" "GCT USB4105-GF-A-120" (at 79.77 66.55 0) (effects (font (size 0.9 0.9))))
-		(property "Footprint" "Connector_USB:USB_C_Receptacle_GCT_USB4105-xx-A_16P_TopMnt_Horizontal" (at 64.77 82.55 0) (effects (font (size 0.9 0.9)) (hide yes)))
+		(property "Footprint" "ENKU:USB4105_EXISTING_LANDS_SHIELD_S" (at 64.77 82.55 0) (effects (font (size 0.9 0.9)) (hide yes)))
 		(property "Datasheet" "~" (at 64.77 82.55 0) (effects (font (size 0.9 0.9)) (hide yes)))
 		(property "Description" "GCT USB4105-GF-A-120" (at 64.77 82.55 0) (effects (font (size 0.9 0.9)) (hide yes)))
@@
 		(property "Value" "USBLC6-2SC6" (at 114.41 58.93 0) (effects (font (size 0.9 0.9))))
 		(property "Footprint" "ENKU:USBLC6_2SC6_ST_SOT23_6L" (at 105.41 74.93 0) (effects (font (size 0.9 0.9)) (hide yes)))
-		(property "Datasheet" "~" (at 105.41 74.93 0) (effects (font (size 0.9 0.9)) (hide yes)))
+		(property "Datasheet" "https://www.st.com/resource/en/datasheet/usblc6-2.pdf" (at 105.41 74.93 0) (effects (font (size 0.9 0.9)) (hide yes)))
 		(property "Description" "USBLC6-2SC6" (at 105.41 74.93 0) (effects (font (size 0.9 0.9)) (hide yes)))
 		(pin "1")
@@
 		(pin "6")
 		(instances (project "enku-mainboard-r0.1" (path "/10000000-0000-4000-8000-000000000001/73000000-0000-4000-8000-000000000056" (reference "U8") (unit 1))))
+		(property "Manufacturer" "STMicroelectronics" (at 0 0 0) (effects (font (size .8 .8)) (hide yes)))
+		(property "MPN" "USBLC6-2SC6" (at 0 0 0) (effects (font (size .8 .8)) (hide yes)))
+		(property "Assembly" "FIT" (at 0 0 0) (effects (font (size .8 .8)) (hide yes)))
 	)
 	(global_label "USB_DP_CONN" (shape input) (at 93.98 72.39 0) (effects (font (size 0.9 0.9)) (justify right bottom)))
@@
 		(property "Reference" "J7" (at 150.02 118.62 0) (effects (font (size 0.9 0.9))))
 		(property "Value" "Tag-Connect TC2030-IDC-NL" (at 170.02 118.62 0) (effects (font (size 0.9 0.9))))
-		(property "Footprint" "Connector:Tag-Connect_TC2030-IDC-NL_2x03_P1.27mm_Vertical" (at 160.02 134.62 0) (effects (font (size 0.9 0.9)) (hide yes)))
-		(property "Datasheet" "~" (at 160.02 134.62 0) (effects (font (size 0.9 0.9)) (hide yes)))
+		(property "Footprint" "ENKU:TC2030_NL_CONTACTS_PIN1" (at 160.02 134.62 0) (effects (font (size 0.9 0.9)) (hide yes)))
+		(property "Datasheet" "https://www.tag-connect.com/wp-content/uploads/bsk-pdf-manager/2019/12/TC2030-IDC-NL-Datasheet-Rev-B.pdf" (at 160.02 134.62 0) (effects (font (size 0.9 0.9)) (hide yes)))
 		(property "Description" "Factory / debug" (at 160.02 134.62 0) (effects (font (size 0.9 0.9)) (hide yes)))
 		(pin "1")
@@
 		(pin "6")
 		(instances (project "enku-mainboard-r0.1" (path "/10000000-0000-4000-8000-000000000001/73000000-0000-4000-8000-000000000108" (reference "J7") (unit 1))))
+		(property "Assembly" "BARE_PCB" (at 0 0 0) (effects (font (size .8 .8)) (hide yes)))
 	)
 	(global_label "3V3_SYS" (shape input) (at 147.32 132.08 0) (effects (font (size 0.9 0.9)) (justify right bottom)))

Commit message: R130 BAT-REV3: PH2 battery and separate NTC; correct Laird lands and preserve R129
Implement the two-wire battery interface, retain all accepted copper identities, and restore the L2 land/via correction. Add native source/assembly/plot guards, supplier evidence and dimensional studies. Charging temperature, capacity/timer, complete mechanical fit and twenty hole findings remain HOLD; no fabrication or orders.
Parts:
- J5: Assembly (none) -> FIT; MPN (none) -> USB4105-GF-A-120; Manufacturer (none) -> GCT
Changed lines of the file:
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@@
 		(property "Value" "GCT USB4105-GF-A-120" (at 79.77 66.55 0) (effects (font (size 0.9 0.9))))
 		(property "Footprint" "ENKU:USB4105_EXISTING_LANDS_SHIELD_S" (at 64.77 82.55 0) (effects (font (size 0.9 0.9)) (hide yes)))
-		(property "Datasheet" "~" (at 64.77 82.55 0) (effects (font (size 0.9 0.9)) (hide yes)))
+		(property "Datasheet" "https://gct.co/connector/usb4105" (at 64.77 82.55 0) (effects (font (size 0.9 0.9)) (hide yes)))
 		(property "Description" "GCT USB4105-GF-A-120" (at 64.77 82.55 0) (effects (font (size 0.9 0.9)) (hide yes)))
 		(pin "A1")
@@
 		(pin "S")
 		(instances (project "enku-mainboard-r0.1" (path "/10000000-0000-4000-8000-000000000001/73000000-0000-4000-8000-000000000001" (reference "J5") (unit 1))))
+		(property "Manufacturer" "GCT" (at 0 0 0) (effects (font (size .8 .8)) (hide yes)))
+		(property "MPN" "USB4105-GF-A-120" (at 0 0 0) (effects (font (size .8 .8)) (hide yes)))
+		(property "Assembly" "FIT" (at 0 0 0) (effects (font (size .8 .8)) (hide yes)))
 	)
 	(global_label "GND" (shape input) (at 46.99 73.66 0) (effects (font (size 0.9 0.9)) (justify right bottom)))

Commit message: R134 working checkpoint: real USB4215 replacement and GPIO charger control; ten routes pending, NO FAB
Parts:
- J5: value GCT USB4105-GF-A-120 -> GCT USB4215-03-A; footprint ENKU:USB4105_EXISTING_LANDS_SHIELD_S -> ENKU:USB4215_03_A_GCT_REVA; MPN USB4105-GF-A-120 -> USB4215-03-A
Changed lines of the file:
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@@
 	(symbol (lib_id "ENKU:USB_C_16P") (at 64.77 82.55 0) (unit 1) (exclude_from_sim no) (in_bom yes) (on_board yes) (dnp no)
 		(property "Reference" "J5" (at 49.77 66.55 0) (effects (font (size 0.9 0.9))))
-		(property "Value" "GCT USB4105-GF-A-120" (at 79.77 66.55 0) (effects (font (size 0.9 0.9))))
-		(property "Footprint" "ENKU:USB4105_EXISTING_LANDS_SHIELD_S" (at 64.77 82.55 0) (effects (font (size 0.9 0.9)) (hide yes)))
-		(property "Datasheet" "https://gct.co/connector/usb4105" (at 64.77 82.55 0) (effects (font (size 0.9 0.9)) (hide yes)))
-		(property "Description" "GCT USB4105-GF-A-120" (at 64.77 82.55 0) (effects (font (size 0.9 0.9)) (hide yes)))
+		(property "Value" "GCT USB4215-03-A" (at 79.77 66.55 0) (effects (font (size 0.9 0.9))))
+		(property "Footprint" "ENKU:USB4215_03_A_GCT_REVA" (at 64.77 82.55 0) (effects (font (size 0.9 0.9)) (hide yes)))
+		(property "Datasheet" "https://gct.co/files/drawings/USB4215.pdf" (at 64.77 82.55 0) (effects (font (size 0.9 0.9)) (hide yes)))
+		(property "Description" "R134 lower3.16mm USB2.0 data receptacle;no locating pegs;4plated shell slots;assembly HOLD" (at 64.77 82.55 0) (effects (font (size 0.9 0.9)) (hide yes)))
 		(pin "A1")
 		(pin "A4")
@@
 		(instances (project "enku-mainboard-r0.1" (path "/10000000-0000-4000-8000-000000000001/73000000-0000-4000-8000-000000000001" (reference "J5") (unit 1))))
 		(property "Manufacturer" "GCT" (at 0 0 0) (effects (font (size .8 .8)) (hide yes)))
-		(property "MPN" "USB4105-GF-A-120" (at 0 0 0) (effects (font (size .8 .8)) (hide yes)))
+		(property "MPN" "USB4215-03-A" (at 0 0 0) (effects (font (size .8 .8)) (hide yes)))
 		(property "Assembly" "FIT" (at 0 0 0) (effects (font (size .8 .8)) (hide yes)))
 	)

Commit message: R137: restore11 fabrication layers, printable silk and explicit R67 DNP stencil; native25 scopes and13 rejection cases; NO FAB
Parts:
- R67: footprint ENKU:R_RC0603_YAGEO_REFLOW -> ENKU:R_RC0603_YAGEO_REFLOW_DNP_NO_PASTE
Changed lines of the file:
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@@
 		(property "Reference" "R67" (at 63.58 128.78 0) (effects (font (size 0.9 0.9))))
 		(property "Value" "0R DNP" (at 73.58 128.78 0) (effects (font (size 0.9 0.9))))
-		(property "Footprint" "ENKU:R_RC0603_YAGEO_REFLOW" (at 68.58 144.78 0) (effects (font (size 0.9 0.9)) (hide yes)))
+		(property "Footprint" "ENKU:R_RC0603_YAGEO_REFLOW_DNP_NO_PASTE" (at 68.58 144.78 0) (effects (font (size 0.9 0.9)) (hide yes)))
 		(property "Datasheet" "https://yageogroup.com/content/datasheet/asset/file/PYU-RC_GROUP_51_ROHS_L" (at 68.58 144.78 0) (effects (font (size 0.9 0.9)) (hide yes)))
 		(property "Description" "0R DNP" (at 68.58 144.78 0) (effects (font (size 0.9 0.9)) (hide yes)))
