File: hardware/mainboard/r144/kicad/enku-mainboard-r0.1.kicad_pcb (KiCad board)
At the start: 4 copper layers, 59 x 101 mm, 134 parts, among them J1 1S LiPo PCM / PH-2, J2 Hirose DM3AT-SF-PEJM5, J3 FH34SRJ-24S-0.5SH(50), J5 GCT USB4215-03-A, J7 Tag-Connect TC2030-IDC-NL, J8 External cell NTC / hand sold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, Q1 IRLML6346TRPBF, Q2 AO3401A, SW1 MK-12C03-G015, SW2 BOOT / RECOVERY, SW3 TL1016AAF160QG, SW4 TL1016AAF160QG, SW5 TL1016AAF160QG, SW6 TL1016AAF160QG, U1 ESP32-S3-WROOM-1-N16R8, U10 TLV3012BIDBVR, U11 TLV803EA30DBZR, U3 BQ24072TRGTR, U4 TPS63802DLAR, U5 BMI270, U8 USBLC6-2SC6, U9 TMUX1101DBVR

Commit message: hardware(r144): route precision reset and PWM supply, fix rule compilation; native checks zero, independent review pending
Parts:
- added C40: 100nF, ENKU:C_CC0603_YAGEO_REFLOW_TRANSFER, F.Cu at (46.0, 71.2)
- added C41: 1nF 50V, ENKU:C_CC0603_YAGEO_REFLOW_TRANSFER, F.Cu at (44.5, 63.9)
- added R95: 16.5k 0.1% 10ppm, ENKU:R_RT0603_YAGEO_REFLOW, F.Cu at (44.5, 65.4)
- added R96: 10k 0.1% 10ppm, ENKU:R_RT0603_YAGEO_REFLOW, F.Cu at (41.5, 66.5)
- added R97: 0R, ENKU:R_RC0603_YAGEO_REFLOW, F.Cu at (63.0, 90.4)
- added R98: 402R 0.1% 10ppm, ENKU:R_RT0603_YAGEO_REFLOW, F.Cu at (59.6, 84.8)
- added R99: 0R, ENKU:R_RC0603_YAGEO_REFLOW_DNP_NO_PASTE, F.Cu at (58.4, 97.4)
- R15: value 4.99k 0.1% 10ppm -> 5.11k 0.1% 10ppm
- U11: value TLV803EA30DBZR -> TPS389001DSER; footprint ENKU:TLV803E_TI_DBZ0003A -> ENKU:TPS3890_TI_DSE0006A_SMD_LEFT
- moved C15 5.81 mm to (46.0, 69.2)
- moved U11 5.48 mm to (44.5, 67.5)
Connections:
- R14 pad 1: 3V3_SYS -> REG_FB_TOP
- U11 pad 1: GND -> RESET_SENSE
- U11 pad 2: ESP_EN -> GND
- U4 pad 2: GND -> REG_MODE
Routing:
- net REG_MODE: track 0.00 -> 17.3 mm, vias 0 -> 3
- net GND: track 332.8 -> 347.1 mm, vias 119 -> 120
- net ESP_EN: track 50.8 -> 63.4 mm, vias 5 -> 7
- net 3V3_SYS: track 448.6 -> 461.1 mm, vias 31 -> 34
- net RESET_SENSE: track 0.00 -> 8.12 mm
- net REG_FB_TOP: track 0.00 -> 6.16 mm, vias 0 -> 2
- net RESET_CT: track 0.00 -> 4.65 mm
