File: hardware/mainboard/r144/kicad/connectors.kicad_sch (KiCad schematic)
At the start: 10 parts, among them J5 GCT USB4215-03-A, J7 Tag-Connect TC2030-IDC-NL, U8 USBLC6-2SC6

Commit message: R144: synchronize schematic titles and confirmed panel annotation; correct informational divider current
Other:
- title: ENKU R143 — External connectors -> ENKU R144 — External connectors
Changed lines of the file:
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@@
 	(paper "A3")
 	(title_block
-		(title "ENKU R143 — External connectors")
-		(date "2026-10-14")
+		(title "ENKU R144 — External connectors")
+		(date "2026-10-15")
 		(rev "R144 - ENGINEERING / NO FAB")
 		(company "ENKU")
